File: PCB_design/PCB_STM32_custom_board/PCB_STM32_custom_board.kicad_sch (KiCad schematic)
At the start: 82 parts, among them J1 Taster, J10 Add-ons, J11 Akku_pins, J12 PowerTaster_pins, J13 USB_B_Micro, J2 Green_LED, J3 Blue_LED, J4 Red_LED, J5 ToF_pins, J6 IMU_pins, J7 Encoder_pins, J8 SWD_pins, J9 Laser_pins, Q1 AO3400A, SW1 SW_SPDT, U1 STM32F446RET6, U3 SIMPLEFOCMINI BRUSHLESS DC MO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, U4 LDO40LPU33RY, U6 Waveshare DC-DC Buck Mini Mod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, U8 USB-C BMS Li-on Batterie Lade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, Y1 16MHz

Commit message: new PCB custom board folder
Parts:
- removed TP10: DRIVER_IN1, symbol Connector:TestPoint
- removed TP11: DRIVER_IN2, symbol Connector:TestPoint
- removed TP12: DRIVER_IN3, symbol Connector:TestPoint
- removed TP13: DRIVER_FAULT, symbol Connector:TestPoint
- removed TP14: DRIVER_EN, symbol Connector:TestPoint
- removed U3: SIMPLEFOCMINI BRUSHLESS DC MOTOR - DRI0058, bachelorarbeit:SIMPLEFOCMINI BRUSHLESS DC MOTOR - DRI0058, symbol bachelorarbeit:SimpleFOCmini_FOC_Brushless_DC_Motor_Driver_Board_-_DRI0058
- removed U6: Waveshare DC-DC Buck Mini Module, bachelorarbeit:WAVESHARE_DC_DC_CONVERTER, symbol bachelorarbeit:Waveshare_DC-DC_Buck_Mini_Module,_bi
- removed U8: USB-C BMS Li-on Batterie Lademodul, symbol bachelorarbeit:USB-C_BMS_Li-on_Batterie_Lademodul_3S_
- added R14: 1k5, Resistor_SMD:R_0402_1005Metric, symbol Device:R
- added U2: USB-C BMS Li-on Batterie Lademodul, bachelorarbeit:USB-C BMS Li-on Batterie Lademodul 3S 4.5V-15V 18W 3A, symbol bachelorarbeit:USB-C_BMS_Li-on_Batterie_Lademodul
- added U3: Waveshare DC-DC Buck Mini Module, bachelorarbeit:WAVESHARE_DC_DC_CONVERTER, symbol bachelorarbeit:Waveshare_DC-DC_Buck_Mini_Module,_bi
- added U6: SIMPLEFOCMINI BRUSHLESS DC MOTOR - DRI0058, bachelorarbeit:SIMPLEFOCMINI BRUSHLESS DC MOTOR - DRI0058, symbol bachelorarbeit:SimpleFOCmini_FOC_Brushless_DC_Motor_Driver_Board_-_DRI0058
- C13: footprint (none) -> Capacitor_SMD:C_0402_1005Metric
- C18: value 470u -> 100u; footprint (none) -> Capacitor_THT:CP_Radial_D6.3mm_P2.50mm
- D1, D2: footprint (none) -> Diode_SMD:D_SMA
- F1: footprint (none) -> Fuse:Fuse_Bourns_MF-RHT200
- H1, H2, H3, H4: footprint (none) -> MountingHole:MountingHole_2.2mm_M2
- J1, J2, J3, J4, J9: footprint (none) -> Connector_JST:JST_PH_B2B-PH-K_1x02_P2.00mm_Vertical
- J10: footprint (none) -> Connector_PinHeader_2.54mm:PinHeader_1x07_P2.54mm_Vertical
- J11, J12: footprint (none) -> Connector_JST:JST_EH_B2B-EH-A_1x02_P2.50mm_Vertical
- J13: footprint Connector_USB:USB_Micro-B_Wuerth_614105150721_Vertical -> Connector_USB:USB_Micro-B_Wuerth_629105150521
- J5: footprint (none) -> Connector_JST:JST_PH_B5B-PH-K_1x05_P2.00mm_Vertical
- J6: footprint (none) -> Connector_JST:JST_PH_B6B-PH-K_1x06_P2.00mm_Vertical
- J8: footprint (none) -> Connector_PinHeader_2.00mm:PinHeader_1x05_P2.00mm_Vertical
- R1, R10, R11, R2, R3, R4, R6, R7: footprint (none) -> Resistor_SMD:R_0402_1005Metric
- R12, R13, R8, R9: footprint Resistor_SMD:R_0402_1005Metric -> Resistor_THT:R_Axial_DIN0207_L6.3mm_D2.5mm_P7.62mm_Horizontal; now not fitted
- SW1: footprint Button_Switch_THT:SW_TH_Tactile_Omron_B3F-112x -> Button_Switch_SMD:SW_SPDT_PCM12
- TP1, TP15, TP19, TP2, TP20, TP3, TP4, TP5, TP6, TP7, TP8, TP9: footprint (none) -> TestPoint:TestPoint_Keystone_5000-5004_Miniature
- TP16, TP17, TP18: footprint (none) -> TestPoint:TestPoint_Bridge_Pitch2.0mm_Drill0.7mm
Connections:
- net +3V3: now also R14.1
- net +5V: now also U3.5 (VOUT)
- net +VDC: now also U3.1 (VIN), U6.11 (VCC)
- net BAT-: now also U2.2 (B-)
- net DRIVER_EN: now also U6.5 (EN)
- net DRIVER_FAULT: now also U6.10 (FAULT)
- net DRIVER_IN1: now also U6.2 (IN1)
- net DRIVER_IN2: now also U6.3 (IN2)
- net DRIVER_IN3: now also U6.4 (IN3)
- net DRIVER_RESET: now also U6.8 (RESET)
- net DRIVER_SLEEP: now also U6.9 (SLEEP)
- net GND: now also U2.4 (VOUT-), U3.3 (GND), U3.7 (VOUT), U6.1 (GND), U6.12 (GND), U6.7 (GND)
- net USB_D+: now also R14.2
- net at D3.1 (K), F1.2: now also U2.1 (B+)
- net at J12.2 (Pin_2): now also U2.3 (VOUT+)
- no-connect marks 28 -> 34
Other:
- note added: "Prototype 4.5 STM32 PCB"
- note removed: "Prototype 4 STM32 PCB"
- title: Prototype 4 STM32 PCB  -> Prototype 4.5 STM32 PCB 
- moved on the sheet: TP15, TP16, TP17, TP18, TP19, TP20
