File: PCB_design/PCB_STM32_custom_board/PCB_STM32_custom_board.kicad_pcb (KiCad board)
At the start: 2 copper layers, 2.2 x 17.4 mm, 78 parts, among them J1 Taster, J10 Add-ons, J11 Akku_pins, J12 PowerTaster_pins, J13 USB_B_Micro, J2 Green_LED, J3 Blue_LED, J4 Red_LED, J5 ToF_pins, J6 IMU_pins, J7 Encoder_pins, J8 SWD_pins, J9 Laser_pins, Q1 AO3400A, SW1 SW_SPDT, U1 STM32F446RET6, U2 USB-C BMS Li-on Batterie Lade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, U3 Waveshare DC-DC Buck Mini Mod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, U4 LDO40LPU33RY, U6 SIMPLEFOCMINI BRUSHLESS DC MO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, Y1 16MHz

Commit message: updated pcb design
Parts:
- Add - ons: renamed from J10
- moved TP16 33.5 mm to (152.2, 113.9), turned to 0 degrees
- moved R4 33.5 mm to (200.2, 86.9), turned to 0 degrees
- moved U6 29.1 mm to (114.7, 109.9)
- moved R_LED 27.8 mm to (199.7, 83.7), turned to 90 degrees
- moved SWD 27.8 mm to (191.2, 84.7)
- moved TP18 27.5 mm to (183.7, 87.9)
- moved TP20 26.7 mm to (187.9, 99.4)
- moved TP17 26.6 mm to (188.9, 87.9)
- moved F1 26.1 mm to (155.2, 97.7)
- moved Add - ons 25.8 mm to (164.3, 129.7)
- moved C15 25.4 mm to (158.8, 106.0)
- moved C19 25.4 mm to (181.2, 107.0)
- moved C4 25.4 mm to (173.0, 107.8)
- moved C5 25.4 mm to (179.3, 107.8)
- moved C6 25.4 mm to (168.7, 97.4)
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- renumbered J11 to Akku, J3 to B_LED, J7 to Encoder, J2 to G_LED, J6 to IMU, J9 to Laser, J12 to Power_Taster, J4 to R_LED, J8 to SWD, J1 to Taster, J5 to ToF
Other:
- board outline removed
